File: PCB_PROJECT.kicad_pcb (KiCad board)
At the start: 2 copper layers, 45 parts, among them J1 USB_C_Receptacle_USB2.0_16P, J2 Conn_01x16_Socket, J3 Conn_01x16_Socket, J4 Conn_PIC_ICSP_ICD, SW1 SW_Push, U1 ATmega328P-A, U2 LM1117DT-ADJ, U3 FT232RL, Y1 16Mhz

Commit message: placing updates
Parts:
- moved FB1 49.2 mm to (130.4, 78.7)
- moved J4 44.9 mm to (175.3, 111.8)
- moved C10 44.1 mm to (133.8, 81.3)
- moved C15 44.1 mm to (133.8, 83.8)
- moved C9 44.1 mm to (133.8, 78.8)
- moved C7 39.2 mm to (150.6, 111.8)
- moved R10 39.2 mm to (154.1, 121.5)
- moved R7 39.2 mm to (154.1, 115.5)
- moved D3 39.2 mm to (152.1, 106.5)
- moved D4 39.2 mm to (152.1, 108.5)
- moved R5 39.2 mm to (154.1, 111.5)
- moved R6 39.2 mm to (154.1, 113.5)
- moved R8 39.2 mm to (154.1, 117.5)
- moved R9 39.2 mm to (154.1, 119.5)
- moved F1 29.0 mm to (124.5, 78.7)
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